File: KiCad Project Files/Switch Matrix.kicad_sch (KiCad schematic)
At the start: 0 parts

Commit message: Finish schematic, annotate footprints, start pcb creation
Parts:
- added D1, D10, D11, D12, D13, D14, D15, D16, D17, D18, D19, D2, D20, D21, D22, D23, D24, D25, D26, D27, D28, D29, D3, D30, D31, D32, D33, D34, D35, D36, D37, D38, D4, D5, D6, D7, D8, D9: D_Small, Diode_SMD:D_SOD-123, symbol Device:D_Small
- added MX1, MX10, MX11, MX13, MX14, MX15, MX16, MX17, MX18, MX20, MX21, MX22, MX24, MX25, MX26, MX27, MX28, MX29, MX30, MX31, MX32, MX33, MX34, MX36, MX37, MX38, MX5, MX6, MX7, MX8, MX9: MX-NoLED, MX_Only:MXOnly-1U-NoLED, symbol cipulot_parts:MX-NoLED
- added MX12, MX2, MX4: MX-NoLED, MX_Only:MXOnly-1.25U-NoLED, symbol cipulot_parts:MX-NoLED
- added MX19, MX23: MX-NoLED, MX_Only:MXOnly-1.75U-NoLED, symbol cipulot_parts:MX-NoLED
- added MX3, MX35: MX-NoLED, MX_Only:MXOnly-1.5U-NoLED, symbol cipulot_parts:MX-NoLED
Connections:
- new net: D19.2 (A), MX19.2 (ROW)
- new net: D35.2 (A), MX35.2 (ROW)
- new net: D37.2 (A), MX37.2 (ROW)
- new net: D32.2 (A), MX32.2 (ROW)
- new net: D20.2 (A), MX20.2 (ROW)
- new net: D34.2 (A), MX34.2 (ROW)
- new net: D3.2 (A), MX3.2 (ROW)
- new net: D30.2 (A), MX30.2 (ROW)
- new net: D17.2 (A), MX17.2 (ROW)
- new net: D33.2 (A), MX33.2 (ROW)
- new net: D21.2 (A), MX21.2 (ROW)
- new net: D11.2 (A), MX11.2 (ROW)
- new net: D18.2 (A), MX18.2 (ROW)
- new net: D5.2 (A), MX5.2 (ROW)
- new net: D26.2 (A), MX26.2 (ROW)
- new net: D36.2 (A), MX36.2 (ROW)
- new net: D27.2 (A), MX27.2 (ROW)
- new net: D16.2 (A), MX16.2 (ROW)
- new net: D1.2 (A), MX1.2 (ROW)
- new net: D23.2 (A), MX23.2 (ROW)
- new net: D28.2 (A), MX28.2 (ROW)
- new net: D24.2 (A), MX24.2 (ROW)
- new net: D4.2 (A), MX4.2 (ROW)
- new net: D29.2 (A), MX29.2 (ROW)
- new net: D38.2 (A), MX38.2 (ROW)
- new net: D13.2 (A), MX13.2 (ROW)
- new net: D14.2 (A), MX14.2 (ROW)
- new net: D22.2 (A), MX22.2 (ROW)
- new net: D31.2 (A), MX31.2 (ROW)
- new net: D12.2 (A), MX12.2 (ROW)
- new net: D6.2 (A), MX6.2 (ROW)
- new net: D9.2 (A), MX9.2 (ROW)
- new net: D8.2 (A), MX8.2 (ROW)
- new net: D25.2 (A), MX25.2 (ROW)
- new net: D7.2 (A), MX7.2 (ROW)
- new net: D15.2 (A), MX15.2 (ROW)
- new net: D2.2 (A), MX2.2 (ROW)
- new net: D10.2 (A), MX10.2 (ROW)
- new net col0: MX1.1 (COL), MX2.1 (COL), MX3.1 (COL), MX4.1 (COL)
- new net col1: MX5.1 (COL), MX6.1 (COL), MX7.1 (COL), MX8.1 (COL)
- new net col2: MX10.1 (COL), MX11.1 (COL), MX12.1 (COL), MX9.1 (COL)
- new net col3: MX13.1 (COL), MX14.1 (COL), MX15.1 (COL)
- new net col4: MX16.1 (COL), MX17.1 (COL), MX18.1 (COL), MX19.1 (COL)
- new net col5: MX20.1 (COL), MX21.1 (COL), MX22.1 (COL), MX23.1 (COL)
- new net col6: MX24.1 (COL), MX25.1 (COL), MX26.1 (COL)
- new net col7: MX27.1 (COL), MX28.1 (COL), MX29.1 (COL), MX30.1 (COL)
- new net col8: MX31.1 (COL), MX32.1 (COL), MX33.1 (COL), MX34.1 (COL)
- new net col9: MX35.1 (COL), MX36.1 (COL), MX37.1 (COL), MX38.1 (COL)
- new net row0: D1.1 (K), D13.1 (K), D16.1 (K), D20.1 (K), D24.1 (K), D27.1 (K), D31.1 (K), D35.1 (K), D5.1 (K), D9.1 (K)
- new net row1: D10.1 (K), D14.1 (K), D17.1 (K), D2.1 (K), D21.1 (K), D25.1 (K), D28.1 (K), D32.1 (K), D36.1 (K), D6.1 (K)
- new net row2: D11.1 (K), D15.1 (K), D18.1 (K), D22.1 (K), D26.1 (K), D29.1 (K), D3.1 (K), D33.1 (K), D37.1 (K), D7.1 (K)
- new net row3: D12.1 (K), D19.1 (K), D23.1 (K), D30.1 (K), D34.1 (K), D38.1 (K), D4.1 (K), D8.1 (K)

Commit message: Finish PCB and create production files
Parts:
- MX36: footprint MX_Only:MXOnly-1U-NoLED -> MX_Only:MXOnly-1.25U-NoLED
Changed lines of the file:
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@@
       (effects (font (size 0.508 0.508)))
     )
-    (property "Footprint" "MX_Only:MXOnly-1U-NoLED" (id 2) (at 189.865 67.945 0)
+    (property "Footprint" "MX_Only:MXOnly-1.25U-NoLED" (id 2) (at 189.865 67.945 0)
       (effects (font (size 1.524 1.524)) hide)
     )
