File: KiCad Project Files/shortiepie2040.kicad_pcb (KiCad board)
At the start: 2 copper layers, 107 parts, among them J1 SM04B, J2 SWD, SW1 Reset, U1 RP2040, U2 W25Q128JVS, U3 XC6206PxxxMR, U4 PRTR5V0U2X, Y1 12MHz

Commit message: Finish PCB and create production files
Parts:
- removed F1: 500mA, Fuse:Fuse_0805_2012Metric
- removed U4: PRTR5V0U2X, random-keyboard-parts:SOT143B
- C_1V-Decoup1, C_1V-Decoup2, C_1V-Decoup3, C_3V-Decoup1, C_3V-Decoup2, C_3V-Decoup3, C_3V-Decoup4, C_3V-Decoup5, C_3V-Decoup6, C_3V-Decoup7, C_3V-Decoup8, C_3V-Decoup9, C_Crystal1, C_Crystal2, C_Flash1, C_LD1, C_LD2, D1, D10, D11, D12, D13, D14, D15, D16, D17, D18, D19, D2, D20, D21, D22, D23, D24, D25, D26, D27, D28, D29, D3, D30, D31, D32, D33, D34, D35, D36, D37, D38, D4, D5, D6, D7, D8, D9, J1, J2, R_Crystal1, R_DATA1, R_DATA2, R_Flash1, R_RST1, SW1, U2, U3, Y1: moved to B.Cu
- MX36: footprint MX_Only:MXOnly-1U-NoLED -> MX_Only:MXOnly-1.25U-NoLED
- U1: footprint Package_DFN_QFN:QFN-56-1EP_7x7mm_P0.4mm_EP3.2x3.2mm -> cipulot_parts:RP2040-QFN-56; moved to B.Cu
- moved J2 210.1 mm to (46.8, 76.0), turned to 180 degrees
- moved D37 207.8 mm to (238.6, 93.9), turned to 90 degrees
- moved D38 196.0 mm to (238.6, 113.0), turned to 90 degrees
- moved D35 187.9 mm to (233.8, 55.8), turned to 90 degrees
- moved D31 185.5 mm to (210.0, 55.8), turned to 90 degrees
- moved MX35 181.9 mm to (230.7, 55.3)
- moved D28 173.8 mm to (195.7, 74.8), turned to 90 degrees
- moved D33 170.2 mm to (219.5, 93.9), turned to 90 degrees
- moved D36 169.8 mm to (236.2, 74.8), turned to 90 degrees
- moved D34 167.7 mm to (219.5, 113.0), turned to 90 degrees
- moved D32 158.5 mm to (214.7, 74.8), turned to 90 degrees
- moved D24 152.1 mm to (171.9, 55.8), turned to 90 degrees
- moved D27 151.1 mm to (190.9, 55.8), turned to 90 degrees
- moved D25 148.9 mm to (176.6, 74.8), turned to 90 degrees
- moved D30 147.5 mm to (200.4, 113.0), turned to 90 degrees
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Routing:
- net row1: track 0.00 -> 239.0 mm, vias 0 -> 7
- net col9: track 0.00 -> 236.3 mm
- net row3: track 0.00 -> 224.3 mm, vias 0 -> 2
- net col8: track 0.00 -> 218.6 mm
- net row0: track 0.00 -> 214.5 mm, vias 0 -> 4
- net col7: track 0.00 -> 200.0 mm
- net row2: track 0.00 -> 197.7 mm, vias 0 -> 2
- net col5: track 0.00 -> 155.0 mm
- net col6: track 0.00 -> 148.3 mm
- net col4: track 0.00 -> 135.4 mm
- net +3V3: track 0.00 -> 109.0 mm, vias 0 -> 5
- net col2: track 0.00 -> 91.0 mm
- net col3: track 0.00 -> 90.4 mm
- net col0: track 0.00 -> 77.4 mm, vias 0 -> 2
- net col1: track 0.00 -> 74.3 mm, vias 0 -> 2
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- added copper zone on B.Cu, net +1V1
- added copper zone on B.Cu, net +3V3
- added copper zone on B.Cu, net GND
- added copper zone on F.Cu, net GND
Other:
- board outline added: 200 x 81 mm
