File: KiCad Project Files/Hotswap PCB/cutiepie2040-hotswap.kicad_pcb (KiCad board)
At the start: 2 copper layers, 200 x 81 mm, 109 parts, among them J1 SM04B-SRSS-TB(LF)(SN), J2 SWD, SW1 BOOTSEL, SW2 RESET, U1 RP2040, U2 W25Q128JVS, U3 XC6206P332MR, Y1 12MHz

Commit message: Added standard stagger hotswap PCB and moved column vias in uniform stagger hotswap PCB outside of solder pads to reduce fabrication cost.
Routing:
- net col9: track 252.7 -> 260.5 mm
- net col8: track 273.3 -> 281.0 mm
- net col7: track 291.6 -> 299.4 mm
- net col0: track 79.0 -> 86.8 mm
- net col5: track 149.5 -> 157.3 mm
- net col4: track 160.1 -> 166.7 mm, vias 7 -> 6
- net col6: track 143.5 -> 149.4 mm
- net col3: track 84.8 -> 90.6 mm
- net col1: track 97.2 -> 101.2 mm
- net col2: track 88.5 -> 91.1 mm
- net Net-(R_Flash1-Pad1): track 41.6 -> 43.0 mm
