File: Baconspoon_Hotswap_and_BLE_PCBs/dual-stagger-hotswap-pcb/MCU-hotswap.kicad_sch (KiCad schematic)
At the start: 32 parts, among them J1 SM04B-SRSS-TB(LF)(SN), J2 SWD, SW1 BOOTSEL, SW2 RESET, U1 RP2040, U2 W25Q128JVS, U3 XC6206P332MR, Y1 12MHz

Commit message: Updated fabrication files for dual-stagger and ortho PCBs and plates. Added stabilizer support for dual-stagger ISO P-key. Updated readme. Updated part mumbers in BOMs and corrected position files. Added KLEs for PCB layouts.
Parts:
- added H2: ISO Stabilizer Drill, MX_Only:MXOnly-ISO-NoSwitch, symbol Mechanical:MountingHole
Changed lines of the file:
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@@
+    )
+  )
+  (symbol (lib_id "Mechanical:MountingHole") (at 252.73 26.67 0) (unit 1)
+    (in_bom yes) (on_board yes) (dnp no) (fields_autoplaced)
+    (property "Reference" "H2" (at 255.27 25.4 0)
+      (effects (font (size 1.27 1.27)) (justify left))
+    )
+    (property "Value" "ISO Stabilizer Drill" (at 255.27 27.94 0)
+      (effects (font (size 1.27 1.27)) (justify left))
+    )
+    (property "Footprint" "MX_Only:MXOnly-ISO-NoSwitch" (at 252.73 26.67 0)
+      (effects (font (size 1.27 1.27)) hide)
+    )
+    (property "Datasheet" "~" (at 252.73 26.67 0)
+      (effects (font (size 1.27 1.27)) hide)
+    )
+    (instances
+      (project "cutiepie2040-dual-stagger-hotswap-pcb"
+        (path "/0bc94950-f950-4f48-816a-6d2035325b5b/765009e9-254e-4f76-82ab-4b2221ccc765"
+          (reference "H2") (unit 1)
+        )
+        (path "/0bc94950-f950-4f48-816a-6d2035325b5b/7af0d888-2a70-4b5e-b2c1-ef82dbe86c73"
+          (reference "H1") (unit 1)
+        )
+      )
     )
   )
